File: electronics/mod_1x1_PSU_1xDC_railsplitter/mod_1x1_PSU_1xDC_railsplitter.kicad_pcb (KiCad board)
At the start: 2 copper layers, 42.5 x 46.2 mm, 53 parts, among them J1 module_2x15_left_input, J2 module_2x15_right_input, J3 Jack-DC, J5 Conn_01x02, U1 LD1117, U2 LM317, U3 LM337, U4 LD1117, U5 TLV431

Commit message: fixed last DRC errors
Parts:
- N1: value 20231206 -> 20231208
- moved D6 0.40 mm to (162.4, 75.7)
Changed lines of the file:
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@@
   )
   (footprint "SquantorDiodes:SOD-323-onsemi" (layer "F.Cu")
-    (at 162.4 75.3 90)
+    (at 162.4 75.7 90)
     (descr "SOD-323 on semiconductor")
     (tags "SOD-323")
@@
         (effects (font (size 1 1) (thickness 0.15)) (justify mirror))
     )
-    (fp_text value "20231206" (at 0 0) (layer "B.SilkS")
+    (fp_text value "20231208" (at 0 0) (layer "B.SilkS")
         (effects (font (size 0.8 0.8) (thickness 0.15)) (justify mirror))
     )
@@
   (segment (start 151.9 86.7) (end 151.1 86.7) (width 1) (layer "F.Cu") (net 1))
   (segment (start 178.73 86.7) (end 180.34 85.09) (width 1) (layer "F.Cu") (net 1))
-  (segment (start 161.175 74.525) (end 161.6 74.1) (width 0.6) (layer "F.Cu") (net 2))
+  (segment (start 163.1 74.5) (end 163.5 74.1) (width 0.6) (layer "F.Cu") (net 2))
   (segment (start 152 79.1) (end 148.55 82.55) (width 1) (layer "F.Cu") (net 2))
   (segment (start 179.55 82.55) (end 176.1 79.1) (width 1) (layer "F.Cu") (net 2))
-  (segment (start 162.4 74.1) (end 171.6 74.1) (width 0.6) (layer "F.Cu") (net 2))
+  (segment (start 162.4 74.5) (end 163.1 74.5) (width 0.6) (layer "F.Cu") (net 2))
+  (segment (start 171.6 74.1) (end 172.1 73.6) (width 0.6) (layer "F.Cu") (net 2))
   (segment (start 176.1 79.1) (end 173.3 79.1) (width 1) (layer "F.Cu") (net 2))
-  (segment (start 171.6 74.1) (end 172.1 73.6) (width 0.6) (layer "F.Cu") (net 2))
-  (segment (start 160.2 74.525) (end 161.175 74.525) (width 0.6) (layer "F.Cu") (net 2))
+  (segment (start 161.3 74.5) (end 162.4 74.5) (width 0.6) (layer "F.Cu") (net 2))
+  (segment (start 161.275 74.525) (end 161.3 74.5) (width 0.6) (layer "F.Cu") (net 2))
   (segment (start 148.55 82.55) (end 144.78 82.55) (width 1) (layer "F.Cu") (net 2))
   (segment (start 173.3 79.1) (end 152 79.1) (width 1) (layer "F.Cu") (net 2))
@@
   (segment (start 173.3 76) (end 173.3 79.1) (width 1) (layer "F.Cu") (net 2))
   (segment (start 182.88 82.55) (end 180.34 82.55) (width 1) (layer "F.Cu") (net 2))
-  (segment (start 161.6 74.1) (end 162.4 74.1) (width 0.6) (layer "F.Cu") (net 2))
+  (segment (start 163.5 74.1) (end 171.6 74.1) (width 0.6) (layer "F.Cu") (net 2))
+  (segment (start 160.2 74.525) (end 161.275 74.525) (width 0.6) (layer "F.Cu") (net 2))
   (via (at 172.1 73.6) (size 0.7) (drill 0.3) (layers "F.Cu" "B.Cu") (net 2))
   (via (at 172.7 73) (size 0.7) (drill 0.3) (layers "F.Cu" "B.Cu") (net 2))
@@
   (segment (start 151.1 114.4) (end 153.2 114.4) (width 1) (layer "F.Cu") (net 17))
   (via (at 153.2 114.4) (size 1) (drill 0.6) (layers "F.Cu" "B.Cu") (net 17))
-  (via (at 160.8 114.4) (size 0.9) (drill 0.6) (layers "F.Cu" "B.Cu") (net 17))
+  (via (at 160.8 114.4) (size 1) (drill 0.6) (layers "F.Cu" "B.Cu") (net 17))
   (segment (start 160.8 114.4) (end 153.2 114.4) (width 1) (layer "B.Cu") (net 17))
   (segment (start 155.7 103.2) (end 155.6 103.3) (width 1) (layer "F.Cu") (net 19))
@@
   (segment (start 178.4 79.1) (end 178.4 75.3) (width 1) (layer "F.Cu") (net 24))
   (segment (start 164 93.9) (end 165.2 92.7) (width 0.4) (layer "F.Cu") (net 24))
-  (segment (start 165.1505 77.7) (end 165.2 77.6505) (width 0.8) (layer "F.Cu") (net 24))
   (segment (start 178.77 74.93) (end 180.34 74.93) (width 1) (layer "F.Cu") (net 24))
-  (segment (start 162.4 76.5) (end 162.4 77.3) (width 0.8) (layer "F.Cu") (net 24))
-  (segment (start 162.8 77.7) (end 165.1505 77.7) (width 0.8) (layer "F.Cu") (net 24))
+  (segment (start 162.4 77.3) (end 162.4 76.9) (width 0.8) (layer "F.Cu") (net 24))
+  (segment (start 165.2 77.6505) (end 165.1505 77.7) (width 0.8) (layer "F.Cu") (net 24))
   (segment (start 173.4 95.4) (end 173.4 93.9) (width 1) (layer "F.Cu") (net 24))
   (segment (start 176.9 83.45) (end 176.9 82.8) (width 0.6) (layer "F.Cu") (net 24))
@@
   (segment (start 162.1 93.9) (end 164 93.9) (width 0.4) (layer "F.Cu") (net 24))
   (segment (start 173.4 93.9) (end 173 93.5) (width 1) (layer "F.Cu") (net 24))
-  (segment (start 162.4 77.3) (end 162.8 77.7) (width 0.8) (layer "F.Cu") (net 24))
   (segment (start 165.2 92.7) (end 165.2 91.65) (width 0.4) (layer "F.Cu") (net 24))
   (segment (start 165.3 91.75) (end 165.2 91.65) (width 0.4) (layer "F.Cu") (net 24))
   (segment (start 160.475 99.525) (end 159.6 99.525) (width 0.6) (layer "F.Cu") (net 24))
+  (segment (start 162.8 77.7) (end 162.4 77.3) (width 0.8) (layer "F.Cu") (net 24))
   (segment (start 160.9 99.1) (end 160.475 99.525) (width 0.6) (layer "F.Cu") (net 24))
   (segment (start 173 93.5) (end 173 90.8) (width 1) (layer "F.Cu") (net 24))
   (segment (start 173.9 96.0625) (end 171.4625 98.5) (width 1) (layer "F.Cu") (net 24))
+  (segment (start 165.1505 77.7) (end 162.8 77.7) (width 0.8) (layer "F.Cu") (net 24))
   (segment (start 161.75 99.1) (end 160.9 99.1) (width 0.6) (layer "F.Cu") (net 24))
   (segment (start 178.4 75.3) (end 178.77 74.93) (width 1) (layer "F.Cu") (net 24))
   (segment (start 166.5 91.75) (end 165.3 91.75) (width 0.4) (layer "F.Cu") (net 24))
+  (segment (start 165.2 75.9) (end 165.2 77.6505) (width 0.8) (layer "F.Cu") (net 24))
   (segment (start 161.5 96.025) (end 161.5 94.5) (width 0.4) (layer "F.Cu") (net 24))
-  (segment (start 165.2 75.9) (end 165.2 77.6505) (width 0.8) (layer "F.Cu") (net 24))
   (segment (start 161.5 94.5) (end 162.1 93.9) (width 0.4) (layer "F.Cu") (net 24))
   (via (at 171.6 98.4) (size 0.7) (drill 0.3) (layers "F.Cu" "B.Cu") (net 24))
-  (via (at 178.4 79.1) (size 1.1) (drill 0.8) (layers "F.Cu" "B.Cu") (net 24))
+  (via (at 178.4 79.1) (size 1) (drill 0.6) (layers "F.Cu" "B.Cu") (net 24))
   (via (at 171.6 99.6) (size 0.7) (drill 0.3) (layers "F.Cu" "B.Cu") (net 24))
   (via (at 172.2 95.4) (size 0.7) (drill 0.3) (layers "F.Cu" "B.Cu") (free) (net 24))
@@
   (via (at 172.8 98.4) (size 0.7) (drill 0.3) (layers "F.Cu" "B.Cu") (net 24))
   (via (at 171.6 100.8) (size 0.7) (drill 0.3) (layers "F.Cu" "B.Cu") (net 24))
-  (via (at 165.2 77.6505) (size 1.1) (drill 0.8) (layers "F.Cu" "B.Cu") (net 24))
+  (via (at 165.1505 77.7) (size 1) (drill 0.6) (layers "F.Cu" "B.Cu") (net 24))
   (via (at 172.2 97.8) (size 0.7) (drill 0.3) (layers "F.Cu" "B.Cu") (net 24))
   (via (at 173.4 95.4) (size 0.7) (drill 0.3) (layers "F.Cu" "B.Cu") (net 24))
@@
   (segment (start 150.3 95.4) (end 152.475 97.575) (width 1) (layer "F.Cu") (net 25))
   (segment (start 161.8 92.5) (end 159.5 94.8) (width 0.4) (layer "F.Cu") (net 25))
+  (segment (start 153.2 104.8) (end 153.2 106.32) (width 1) (layer "F.Cu") (net 25))
   (segment (start 159.5 94.8) (end 159.6 94.9) (width 0.6) (layer "F.Cu") (net 25))
   (segment (start 161.8 91.95) (end 161.8 92.5) (width 0.4) (layer "F.Cu") (net 25))
@@
   (segment (start 158 106.32) (end 158 104.8) (width 1) (layer "F.Cu") (net 25))
   (segment (start 159.6 94.9) (end 159.6 96) (width 0.6) (layer "F.Cu") (net 25))
-  (segment (start 153.2 104.8) (end 153.2 106.32) (width 1) (layer "F.Cu") (net 25))
   (segment (start 155.8 99.1) (end 155.8 97.575) (width 1) (layer "F.Cu") (net 25))
   (segment (start 162.45 92.35) (end 162.3 92.5) (width 0.4) (layer "F.Cu") (net 25))
@@
   (via (at 156.3 83.6375) (size 0.7) (drill 0.3) (layers "F.Cu" "B.Cu") (net 25))
   (via (at 156.9 83.0375) (size 0.7) (drill 0.3) (layers "F.Cu" "B.Cu") (net 25))
-  (via (at 153.2 104.8) (size 0.9) (drill 0.6) (layers "F.Cu" "B.Cu") (net 25))
+  (via (at 153.2 104.8) (size 1) (drill 0.6) (layers "F.Cu" "B.Cu") (net 25))
   (via (at 156.9 84.2375) (size 0.7) (drill 0.3) (layers "F.Cu" "B.Cu") (net 25))
   (via (at 156.3 82.4375) (size 0.7) (drill 0.3) (layers "F.Cu" "B.Cu") (net 25))
-  (via (at 158 104.8) (size 0.9) (drill 0.6) (layers "F.Cu" "B.Cu") (net 25))
+  (via (at 158 104.8) (size 1) (drill 0.6) (layers "F.Cu" "B.Cu") (net 25))
   (via (at 157.5 82.4375) (size 0.7) (drill 0.3) (layers "F.Cu" "B.Cu") (net 25))
   (via (at 158.7 83.6375) (size 0.7) (drill 0.3) (layers "F.Cu" "B.Cu") (net 25))
@@
   (segment (start 150.3 95.4) (end 149.4 94.5) (width 1) (layer "B.Cu") (net 25))
   (segment (start 149.4 79.2) (end 149.5 79.1) (width 1) (layer "B.Cu") (net 25))
+  (segment (start 158 104.8) (end 153.2 104.8) (width 1) (layer "B.Cu") (net 25))
   (segment (start 148.95 79.1) (end 147.32 77.47) (width 1) (layer "B.Cu") (net 25))
-  (segment (start 152.1 97.2) (end 152.1 103.7) (width 1) (layer "B.Cu") (net 25))
-  (segment (start 150.3 95.4) (end 152.1 97.2) (width 1) (layer "B.Cu") (net 25))
+  (segment (start 153.2 104.8) (end 152.1 103.7) (width 1) (layer "B.Cu") (net 25))
+  (segment (start 152.1 103.7) (end 152.1 97.2) (width 1) (layer "B.Cu") (net 25))
   (segment (start 177.93 77.47) (end 176.3 79.1) (width 1) (layer "B.Cu") (net 25))
-  (segment (start 158 104.8) (end 153.2 104.8) (width 1) (layer "B.Cu") (net 25))
   (segment (start 151.9 79.1) (end 149.5 79.1) (width 1) (layer "B.Cu") (net 25))
+  (segment (start 152.1 97.2) (end 150.3 95.4) (width 1) (layer "B.Cu") (net 25))
   (segment (start 176.3 79.1) (end 151.9 79.1) (width 1) (layer "B.Cu") (net 25))
-  (segment (start 152.1 103.7) (end 153.2 104.8) (width 1) (layer "B.Cu") (net 25))
   (segment (start 149.5 79.1) (end 148.95 79.1) (width 1) (layer "B.Cu") (net 25))
   (segment (start 168.6 111.1) (end 167.7 112) (width 1) (layer "F.Cu") (net 28))

Commit message: final changes and some extra vias
Parts:
- N1: value 20231208 -> 20231213
Routing:
- net GND: vias 0 -> 3
Changed lines of the file:
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@@
         (effects (font (size 1 1) (thickness 0.15)) (justify mirror))
     )
-    (fp_text value "20231208" (at 0 0) (layer "B.SilkS")
+    (fp_text value "20231213" (at 0 0) (layer "B.SilkS")
         (effects (font (size 0.8 0.8) (thickness 0.15)) (justify mirror))
     )
@@
   (segment (start 151.9 86.7) (end 151.1 86.7) (width 1) (layer "F.Cu") (net 1))
   (segment (start 178.73 86.7) (end 180.34 85.09) (width 1) (layer "F.Cu") (net 1))
+  (via (at 153.2 74.1) (size 0.7) (drill 0.3) (layers "F.Cu" "B.Cu") (free) (net 1))
+  (via (at 153.2 72.6) (size 0.7) (drill 0.3) (layers "F.Cu" "B.Cu") (free) (net 1))
+  (via (at 160.2 69.9) (size 0.7) (drill 0.3) (layers "F.Cu" "B.Cu") (free) (net 1))
   (segment (start 163.1 74.5) (end 163.5 74.1) (width 0.6) (layer "F.Cu") (net 2))
   (segment (start 152 79.1) (end 148.55 82.55) (width 1) (layer "F.Cu") (net 2))
@@
   (segment (start 158.3 76.1) (end 160.175 76.1) (width 0.6) (layer "F.Cu") (net 31))
   (segment (start 160.175 76.1) (end 160.2 76.075) (width 0.6) (layer "F.Cu") (net 31))
-  (segment (start 166.5 89.8) (end 166.2 89.5) (width 0.4) (layer "F.Cu") (net 32))
   (segment (start 165.1 88.4) (end 165.55 88.85) (width 0.4) (layer "F.Cu") (net 32))
   (segment (start 168.4 92.3) (end 168.9 92.8) (width 0.4) (layer "F.Cu") (net 32))
-  (segment (start 166.5 90.05) (end 166.5 89.8) (width 0.4) (layer "F.Cu") (net 32))
   (segment (start 165.55 88.85) (end 166.2 88.85) (width 0.4) (layer "F.Cu") (net 32))
   (segment (start 166.5 90.05) (end 165.3 90.05) (width 0.4) (layer "F.Cu") (net 32))
   (segment (start 165.3 90.05) (end 165.2 90.15) (width 0.4) (layer "F.Cu") (net 32))
   (segment (start 168.15 90.05) (end 166.5 90.05) (width 0.4) (layer "F.Cu") (net 32))
+  (segment (start 166.2 89.3) (end 166.5 89.6) (width 0.4) (layer "F.Cu") (net 32))
   (segment (start 163.1 88.4) (end 165.1 88.4) (width 0.4) (layer "F.Cu") (net 32))
   (segment (start 168.4 90.3) (end 168.15 90.05) (width 0.4) (layer "F.Cu") (net 32))
@@
   (segment (start 168.4 90.8) (end 168.4 92.3) (width 0.4) (layer "F.Cu") (net 32))
   (segment (start 168.4 90.8) (end 168.4 90.3) (width 0.4) (layer "F.Cu") (net 32))
-  (segment (start 166.2 89.5) (end 166.2 88.85) (width 0.4) (layer "F.Cu") (net 32))
+  (segment (start 166.5 89.6) (end 166.5 90.05) (width 0.4) (layer "F.Cu") (net 32))
+  (segment (start 166.2 88.85) (end 166.2 89.3) (width 0.4) (layer "F.Cu") (net 32))
   (segment (start 162.85 87.4) (end 162.85 88.15) (width 0.4) (layer "F.Cu") (net 32))
   (segment (start 162.85 90.05) (end 162.9 90) (width 0.4) (layer "F.Cu") (net 33))
@@
   (segment (start 156.4 71.025) (end 158.3 71.025) (width 0.6) (layer "F.Cu") (net 36))
   (segment (start 154.5 71.025) (end 156.4 71.025) (width 0.6) (layer "F.Cu") (net 36))
-  (segment (start 158.8 98) (end 159.6 98) (width 0.4) (layer "F.Cu") (net 37))
   (segment (start 164.5625 96.2) (end 164.5625 97.2375) (width 0.4) (layer "F.Cu") (net 37))
   (segment (start 160.15 97.8) (end 159.95 98) (width 0.4) (layer "F.Cu") (net 37))
@@
   (segment (start 164.5625 97.2375) (end 164.225 97.575) (width 0.4) (layer "F.Cu") (net 37))
   (segment (start 164.225 97.575) (end 161.5 97.575) (width 0.4) (layer "F.Cu") (net 37))
+  (segment (start 157.925 97.8) (end 157.7 97.575) (width 0.4) (layer "F.Cu") (net 37))
   (segment (start 161.275 97.8) (end 160.15 97.8) (width 0.4) (layer "F.Cu") (net 37))
-  (segment (start 157.7 97.575) (end 158.375 97.575) (width 0.4) (layer "F.Cu") (net 37))
-  (segment (start 158.375 97.575) (end 158.8 98) (width 0.4) (layer "F.Cu") (net 37))
-  (segment (start 159.5 73) (end 160.2 73) (width 0.4) (layer "F.Cu") (net 38))
-  (segment (start 160.2 73) (end 160.9 73) (width 0.4) (layer "F.Cu") (net 38))
-  (segment (start 160.9 73) (end 161.325 72.575) (width 0.4) (layer "F.Cu") (net 38))
+  (segment (start 159.6 98) (end 159.4 97.8) (width 0.4) (layer "F.Cu") (net 37))
+  (segment (start 159.4 97.8) (end 157.925 97.8) (width 0.4) (layer "F.Cu") (net 37))
+  (segment (start 160.2 73) (end 160.4 72.8) (width 0.4) (layer "F.Cu") (net 38))
+  (segment (start 160 72.8) (end 158.525 72.8) (width 0.4) (layer "F.Cu") (net 38))
+  (segment (start 160.2 73) (end 160 72.8) (width 0.4) (layer "F.Cu") (net 38))
   (segment (start 165.2 71.3) (end 165.2 72.4) (width 0.6) (layer "F.Cu") (net 38))
-  (segment (start 161.325 72.575) (end 162.1 72.575) (width 0.4) (layer "F.Cu") (net 38))
-  (segment (start 158.3 72.575) (end 159.075 72.575) (width 0.4) (layer "F.Cu") (net 38))
-  (segment (start 159.075 72.575) (end 159.5 73) (width 0.4) (layer "F.Cu") (net 38))
+  (segment (start 158.525 72.8) (end 158.3 72.575) (width 0.4) (layer "F.Cu") (net 38))
   (segment (start 165.2 72.4) (end 165.025 72.575) (width 0.6) (layer "F.Cu") (net 38))
+  (segment (start 161.875 72.8) (end 162.1 72.575) (width 0.4) (layer "F.Cu") (net 38))
   (segment (start 165.025 72.575) (end 162.1 72.575) (width 0.6) (layer "F.Cu") (net 38))
+  (segment (start 160.4 72.8) (end 161.875 72.8) (width 0.4) (layer "F.Cu") (net 38))
   (segment (start 164.1 87.4) (end 164.75 87.4) (width 0.4) (layer "F.Cu") (net 39))
   (segment (start 163.8 81.3) (end 163.8 87.1) (width 0.4) (layer "F.Cu") (net 39))
