File: electronics/mod_1x1_PSU_1xDC_railsplitter/mod_1x1_PSU_1xDC_railsplitter.kicad_sch (KiCad schematic)
At the start: 53 parts, among them J1 module_2x15_left_input, J2 module_2x15_right_input, J3 Jack-DC, J5 Conn_01x02, U1 LD1117, U2 LM317, U3 LM337, U4 LD1117, U5 TLV431

Commit message: final changes and some extra vias
Parts:
- N1: value 20231208 -> 20231213
Changed lines of the file:
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@@
       (effects (font (size 1.524 1.524)) (justify left))
     )
-    (property "Value" "20231208" (at 19.05 189.23 0)
+    (property "Value" "20231213" (at 19.05 189.23 0)
       (effects (font (size 1.524 1.524)) (justify left))
     )
