File: electronics/ModEleSysV2_1x03_PSU_Batt_symmetrical/ModEleSysV2_1x03_PSU_Batt_symmetrical.kicad_sch (KiCad schematic)
At the start: 18 parts, among them J2 Conn_01x02, J3 Conn_01x02, J4 Conn_01x03, SW1 switch_DPDT, U1 TSC432

Commit message: silk placement done, ready for review
Connections:
- no-connect marks 22 -> 24
Other:
- note added: "Filtering Decoupling"
- moved on the sheet: C2, C3, C4, C5

Commit message: reviewed
Parts:
- C2, C3: footprint SquantorCapacitor:C_0805 -> SquantorCapacitor:C_1206_0805
- N1: value 20240311 -> 20240424
Changed lines of the file:
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@@
       (effects (font (size 1.524 1.524)) (justify left))
     )
-    (property "Value" "20240311" (at 20.32 189.23 0)
+    (property "Value" "20240424" (at 20.32 189.23 0)
       (effects (font (size 1.524 1.524)) (justify left))
     )
@@
       (effects (font (size 1.27 1.27)))
     )
-    (property "Footprint" "SquantorCapacitor:C_0805" (at 60.96 63.8048 0)
+    (property "Footprint" "SquantorCapacitor:C_1206_0805" (at 60.96 63.8048 0)
       (effects (font (size 1.27 1.27)) hide)
     )
@@
       (effects (font (size 1.27 1.27)))
     )
-    (property "Footprint" "SquantorCapacitor:C_0805" (at 60.96 68.8848 0)
-      (effects (font (size 1.27 1.27)) hide)
-    )
+    (property "Footprint" "SquantorCapacitor:C_1206_0805" (at 60.96 68.8848 0)
+      (effects (font (size 1.27 1.27)) hide)
+    )

Commit message: updated versionnumbers
Parts:
- N1: value 20240424 -> 20240426
Changed lines of the file:
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@@
       (effects (font (size 1.524 1.524)) (justify left))
     )
-    (property "Value" "20240424" (at 20.32 189.23 0)
+    (property "Value" "20240426" (at 20.32 189.23 0)
       (effects (font (size 1.524 1.524)) (justify left))
     )
