File: electronics/ModEleSysV2_1x1_PSU_AC_symmetrical/ModEleSysV2_1x1_PSU_AC_symmetrical.kicad_sch (KiCad schematic)
At the start: 30 parts, among them J2 Jack-DC, SW1 switch_DPDT, U1 LM317, U2 LM337

Commit message: preparations for production
Parts:
- N1: value 20240426 -> 20250323
Changed lines of the file:
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@@
 			)
 		)
-		(property "Value" "20240426"
+		(property "Value" "20250323"
 			(at 20.32 189.23 0)
 			(effects
@@
 			)
 		)
-		(property "Description" ""
+		(property "Description" "Power symbol creates a global label with name \"GND\" , ground"
 			(at 72.39 21.59 0)
 			(effects
@@
 			)
 		)
-		(property "Description" ""
+		(property "Description" "Diode"
 			(at 66.04 29.21 0)
 			(effects
@@
 			)
 		)
-		(property "Description" ""
+		(property "Description" "SquMes 30 pin bus using DIN41612 connector"
 			(at 19.05 93.98 0)
 			(effects
@@
 			)
 		)
-		(property "Description" ""
+		(property "Description" "Power symbol creates a global label with name \"GND\" , ground"
 			(at 92.71 17.78 0)
 			(effects
@@
 			)
 		)
-		(property "Description" ""
+		(property "Description" "LM337 3 pin generic variable regulator"
 			(at 90.17 31.75 0)
 			(effects
@@
 			)
 		)
-		(property "Description" ""
+		(property "Description" "Resistor"
 			(at 102.87 21.59 0)
 			(effects
@@
 			)
 		)
-		(property "Description" ""
+		(property "Description" "Resistor"
 			(at 66.04 21.59 0)
 			(effects
@@
 			)
 		)
-		(property "Description" ""
+		(property "Description" "Unpolarized capacitor"
 			(at 50.8 17.78 0)
 			(effects
@@
 			)
 		)
-		(property "Description" ""
+		(property "Description" "Diode"
 			(at 102.87 29.21 0)
 			(effects
@@
 			)
 		)
-		(property "Description" ""
+		(property "Description" "Unpolarized capacitor"
 			(at 102.87 17.78 0)
 			(effects
@@
 			)
 		)
-		(property "Description" ""
+		(property "Description" "Diode"
 			(at 95.25 39.37 0)
 			(effects
@@
 			)
 		)
-		(property "Description" ""
+		(property "Description" "Resistor"
 			(at 102.87 26.67 0)
 			(effects
@@
 			)
 		)
-		(property "Description" ""
+		(property "Description" "Special symbol for telling ERC where power comes from"
 			(at 54.61 59.69 0)
 			(effects
@@
 			)
 		)
-		(property "Description" ""
+		(property "Description" "Power symbol creates a global label with name \"GND\" , ground"
 			(at 76.2 33.02 0)
 			(effects
@@
 			)
 		)
-		(property "Description" ""
+		(property "Description" "Resistor"
 			(at 102.87 24.13 0)
 			(effects
@@
 			)
 		)
-		(property "Description" ""
+		(property "Description" "Special symbol for telling ERC where power comes from"
 			(at 54.61 49.53 0)
 			(effects
@@
 			)
 		)
-		(property "Description" ""
+		(property "Description" "Unpolarized capacitor"
 			(at 46.99 59.69 0)
 			(effects
@@
 	)
 	(symbol
-		(lib_name "SquMes_30pin_2")
 		(lib_id "SquantorConnectorsNamed:SquMes_30pin")
 		(at 19.05 62.23 0)
@@
 			)
 		)
-		(property "Description" ""
+		(property "Description" "SquMes 30 pin bus using DIN41612 connector"
 			(at 19.05 62.23 0)
 			(effects
@@
 			)
 		)
-		(property "Description" ""
+		(property "Description" "Resistor"
 			(at 66.04 26.67 0)
 			(effects
@@
 			)
 		)
-		(property "Description" ""
+		(property "Description" "Unpolarized capacitor"
 			(at 87.63 17.78 0)
 			(effects
@@
 			)
 		)
-		(property "Description" ""
+		(property "Description" "Power symbol creates a global label with name \"GND\" , ground"
 			(at 55.88 17.78 0)
 			(effects
@@
 			)
 		)
-		(property "Description" ""
+		(property "Description" "Polarized capacitor"
 			(at 50.8 54.61 0)
 			(effects
@@
 			)
 		)
-		(property "Description" ""
+		(property "Description" "Special symbol for telling ERC where power comes from"
 			(at 54.61 69.85 0)
 			(effects
@@
 	)
 	(symbol
-		(lib_name "SquMes_30pin_1")
 		(lib_id "SquantorConnectorsNamed:SquMes_30pin")
 		(at 19.05 30.48 0)
@@
 			)
 		)
-		(property "Description" ""
+		(property "Description" "SquMes 30 pin bus using DIN41612 connector"
 			(at 19.05 30.48 0)
 			(effects
@@
 			)
 		)
-		(property "Description" ""
+		(property "Description" "DC Barrel Jack with an internal switch"
 			(at 22.86 129.54 0)
 			(effects
@@
 			)
 		)
-		(property "Description" ""
+		(property "Description" "Power symbol creates a global label with name \"GND\" , ground"
 			(at 25.4 74.93 0)
 			(effects
@@
 			)
 		)
-		(property "Description" ""
+		(property "Description" "Diode"
 			(at 46.99 49.53 0)
 			(effects
@@
 			)
 		)
-		(property "Description" ""
+		(property "Description" "Power symbol creates a global label with name \"GND\" , ground"
 			(at 54.61 57.15 0)
 			(effects
@@
 			)
 		)
-		(property "Description" ""
+		(property "Description" "Polarized capacitor"
 			(at 50.8 64.77 0)
 			(effects
@@
 			)
 		)
-		(property "Description" ""
+		(property "Description" "Fuse"
 			(at 22.86 140.97 0)
 			(effects
@@
 			)
 		)
-		(property "Description" ""
+		(property "Description" "Resistor"
 			(at 66.04 24.13 0)
 			(effects
@@
 			)
 		)
-		(property "Description" ""
+		(property "Description" "Power symbol creates a global label with name \"GND\" , ground"
 			(at 109.22 21.59 0)
 			(effects
@@
 			)
 		)
-		(property "Description" ""
+		(property "Description" "Diode"
 			(at 53.34 39.37 0)
 			(effects
@@
 			)
 		)
-		(property "Description" ""
+		(property "Description" "Mounting Hole without connection"
 			(at 19.05 111.76 0)
 			(effects
@@
 			)
 		)
-		(property "Description" ""
+		(property "Description" "Power symbol creates a global label with name \"GND\" , ground"
 			(at 17.78 140.97 0)
 			(effects
@@
 			)
 		)
-		(property "Description" ""
+		(property "Description" "LM317 3 pin generic variable regulator"
 			(at 53.34 31.75 0)
 			(effects
@@
 			)
 		)
-		(property "Description" ""
+		(property "Description" "Unpolarized capacitor"
 			(at 66.04 17.78 0)
 			(effects
@@
 			)
 		)
-		(property "Description" ""
+		(property "Description" "Diode"
 			(at 46.99 69.85 0)
 			(effects

Commit message: added backplane, updated kicad file versions
Changed lines of the file:
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@@
 (kicad_sch
-	(version 20231120)
+	(version 20250114)
 	(generator "eeschema")
-	(generator_version "8.0")
+	(generator_version "9.0")
 	(paper "A4")
+	(text "ModEleSys connections"
+		(exclude_from_sim no)
+		(at 15.24 119.38 0)
+		(effects
+			(font
+				(size 1.27 1.27)
+			)
+			(justify left bottom)
+		)
+	)
+	(text "Logos and version"
+		(exclude_from_sim no)
+		(at 16.51 194.31 0)
+		(effects
+			(font
+				(size 1.27 1.27)
+			)
+			(justify left bottom)
+		)
+	)
+	(text "Power filter"
+		(exclude_from_sim no)
+		(at 49.53 74.93 0)
+		(effects
+			(font
+				(size 1.27 1.27)
+			)
+			(justify left bottom)
+		)
+	)
+	(text "Power input"
+		(exclude_from_sim no)
+		(at 44.45 147.32 0)
+		(effects
+			(font
+				(size 1.27 1.27)
+			)
+			(justify left bottom)
+		)
+	)
+	(text "Regulators"
+		(exclude_from_sim no)
+		(at 102.87 41.91 0)
+		(effects
+			(font
+				(size 1.27 1.27)
+			)
+			(justify left bottom)
+		)
+	)
 	(junction
 		(at 71.12 26.67)
@@
 		)
 	)
-	(text "ModEleSys connections"
-		(exclude_from_sim no)
-		(at 15.24 119.38 0)
-		(effects
-			(font
-				(size 1.27 1.27)
-			)
-			(justify left bottom)
-		)
-	)
-	(text "Logos and version"
-		(exclude_from_sim no)
-		(at 16.51 194.31 0)
-		(effects
-			(font
-				(size 1.27 1.27)
-			)
-			(justify left bottom)
-		)
-	)
-	(text "Power filter"
-		(exclude_from_sim no)
-		(at 49.53 74.93 0)
-		(effects
-			(font
-				(size 1.27 1.27)
-			)
-			(justify left bottom)
-		)
-	)
-	(text "Power input"
-		(exclude_from_sim no)
-		(at 44.45 147.32 0)
-		(effects
-			(font
-				(size 1.27 1.27)
-			)
-			(justify left bottom)
-		)
-	)
-	(text "Regulators"
-		(exclude_from_sim no)
-		(at 102.87 41.91 0)
-		(effects
-			(font
-				(size 1.27 1.27)
-			)
-			(justify left bottom)
-		)
-	)
 	(label "+aV"
 		(at 25.4 19.05 0)
@@
 		)
 	)
+	(embedded_fonts no)
 )
