File: electronics/ModEleSysV2_1x1_PSU_AC_symmetrical/ModEleSysV2_1x1_PSU_AC_symmetrical.kicad_sch (KiCad schematic)
At the start: 30 parts, among them J2 Jack-DC, SW1 switch_DPDT, U1 LM317, U2 LM337

Commit message: reviewed and updated PCB's
Parts:
- removed SW1: switch_DPDT, SquantorSwitches:PS-22F02, symbol SquantorSwitches:switch_DPDT
- added J3: PINS_2X03, SquantorConnectors:DLL-XHY-6A, symbol SquantorConnectors:PINS_2X03
- C4, C7: value 22u -> 47u
- U1, U2: footprint SquantorIC:TO-252_D-PAK_IRF -> SquantorIC:SOT-223
Connections:
- net AC1_PHASE: now also J3.4
- net AC_NEUT_IN: now also J2.1, J3.1; no longer J2.2
- net AC_PHASE1_IN: now also J2.2, J3.2; no longer J2.1
- net at F1.1: now also J3.3
Other:
- moved on the sheet: C4, C7, F1

Commit message: Updated for production
Parts:
- N1: value 20250323 -> V:20260118
Changed lines of the file:
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@@
 			)
 		)
-		(property "Value" "20250323"
+		(property "Value" "V:20260118"
 			(at 20.32 189.23 0)
 			(effects
