File: electronics/ModEleSysV2_backplane/ModEleSysV2_backplane.kicad_sch (KiCad schematic)
At the start: 38 parts, among them J5 Conn_01x03, J6 Conn_01x03, J7 Conn_02x03_Odd_Even, J9 Conn_02x03_Odd_Even, SW1 switch_DPDT, SW2 switch_DPDT

Commit message: Updated for production
Parts:
- N2: value V:20251015 -> V:20260118
Changed lines of the file:
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@@
 			)
 		)
-		(property "Value" "V:20251015"
+		(property "Value" "V:20260118"
 			(at 158.75 167.64 0)
 			(effects
